Commit message: controllers shaghala inshallah

File: src/abb_package/assembly_environment/urdf/environment.xacro (robot description, xacro)
@@ -11,5 +11,5 @@
         <origin xyz="0 0 0" rpy="0 0 0" />
         <geometry>
-          <mesh filename="package://assembly_environment/meshes/abb_table.STL" />
+          <mesh filename="file://$(find assembly_environment)/meshes/abb_table.STL" />
         </geometry>
         <material name="">
@@ -20,5 +20,5 @@
         <origin xyz="0 0 0" rpy="0 0 0" />
         <geometry>
-          <mesh filename="package://assembly_environment/meshes/abb_table.STL" />
+          <mesh filename="file://$(find assembly_environment)/meshes/abb_table.STL" />
         </geometry>
       </collision>
@@ -33,5 +33,5 @@
         <origin xyz="0 0 0" rpy="0 0 0" />
         <geometry>
-          <mesh filename="package://assembly_environment/meshes/ar4_table.STL" />
+          <mesh filename="file://$(find assembly_environment)/meshes/ar4_table.STL" />
         </geometry>
         <material name="">
@@ -42,5 +42,5 @@
         <origin xyz="0 0 0" rpy="0 0 0" />
         <geometry>
-          <mesh filename="package://assembly_environment/meshes/ar4_table.STL" />
+          <mesh filename="file://$(find assembly_environment)/meshes/ar4_table.STL" />
         </geometry>
       </collision>
@@ -60,5 +60,5 @@
         <origin xyz="0 0 0" rpy="0 0 0" />
         <geometry>
-          <mesh filename="package://assembly_environment/meshes/camera.STL" />
+          <mesh filename="file://$(find assembly_environment)/meshes/camera.STL" />
         </geometry>
         <material name="">
@@ -69,5 +69,5 @@
         <origin xyz="0 0 0" rpy="0 0 0" />
         <geometry>
-          <mesh filename="package://assembly_environment/meshes/camera.STL" />
+          <mesh filename="file://$(find assembly_environment)/meshes/camera.STL" />
         </geometry>
       </collision>

File: src/abb_package/ros2_SimRealRobotControl/ros2srrc_endeffectors/egp64/urdf/egp64_macro.urdf.xacro (robot description, xacro)
@@ -51,8 +51,6 @@
       <inertial>
         <origin xyz="0 0 0" rpy="0 0 ${pi/2}" />
-        <mass value="0.03"/>
-        <inertia ixx="4.09e-06" ixy="0.0" ixz="0.0"
-                iyy="4.09e-06" iyz="0.0"
-                izz="8.00e-06"/>
+        <mass value="0.001" />
+        <inertia ixx="0.001" ixy="0.0" ixz="0.0" iyy="0.001" iyz="0.0" izz="0.001"/>
       </inertial>
     </link>
@@ -70,9 +68,7 @@
     <link name="egp64_gripper_base_link">
       <inertial>
-        <origin xyz="0 0 0" rpy="0 0 0"/>
-        <mass value="0.72"/>
-        <inertia ixx="9.375e-04" ixy="0.0" ixz="0.0"
-                iyy="1.10976e-03" iyz="0.0"
-                izz="3.1926e-04"/>
+        <origin xyz="0 0 0" rpy="0 0 0" />
+        <mass value="0.005" />
+        <inertia ixx="0.001" ixy="0.0" ixz="0.0" iyy="0.001" iyz="0.0" izz="0.001"/>
       </inertial>
       <visual>
@@ -80,6 +76,6 @@
           <mesh filename="file://$(find ros2srrc_endeffectors)/egp64/meshes/egp64_BaseNoAdapter.dae" />
         </geometry>
-        <material name="silver">
-          <color rgba="0.8 0.8 0.8 1"/>
+        <material name="blue">
+          <color rgba="0 0 1 1"/>
         </material>
       </visual>
@@ -88,4 +84,5 @@
           <mesh filename="file://$(find ros2srrc_endeffectors)/egp64/meshes/egp64_BaseNoAdapter.dae" />
         </geometry>
+        <material name="blue"/>
       </collision>
     </link>
@@ -99,8 +96,6 @@
       <inertial>
         <origin xyz="0.01483 -0.00782 0" rpy="0 0 0" />
-        <mass value="0.02"/>
-        <inertia ixx="3.47e-07" ixy="0.0" ixz="0.0"
-                iyy="2.77e-06" iyz="0.0"
-                izz="2.91e-06"/>
+        <mass value="0.002" />
+        <inertia ixx="0.001" ixy="0.0" ixz="0.0" iyy="0.001" iyz="0.0" izz="0.001"/>
       </inertial>
       <visual>
@@ -116,4 +111,5 @@
           <mesh filename="file://$(find ros2srrc_endeffectors)/egp64/meshes/egp64_LeftFingerBase.dae" />
         </geometry>
+        <material name="black" />
       </collision>
     </link>
@@ -121,8 +117,8 @@
       <parent link="egp64_gripper_base_link" />
       <child link="egp64_finger_left_link" />
-      <limit effort="1000" lower="-0.0001" upper="0.027" velocity="0.2"/>
+      <limit effort="1000" lower="-0.001" upper="0.04" velocity="0.2"/>
       <origin xyz="0.01483 -0.00782 0" rpy="0 0 0" />
       <axis xyz="-1 0 0" />
-      <dynamics damping="0.2" friction="0.05"/>
+      <dynamics damping="1.0" friction="1.0"/>
     </joint>
     <!-- LEFT FINGERTIP -->
@@ -130,8 +126,6 @@
       <inertial>
         <origin xyz="0.03869 -0.0005 0.00093" rpy="0 0 0" />
-        <mass value="0.005"/>
-        <inertia ixx="3.71e-08" ixy="0.0" ixz="0.0"
-                iyy="1.77e-07" iyz="0.0"
-                izz="1.93e-07"/>
+        <mass value="0.001" />
+        <inertia ixx="0.001" ixy="0.0" ixz="0.0" iyy="0.001" iyz="0.0" izz="0.001"/>
       </inertial>
       <visual>
@@ -147,4 +141,5 @@
           <mesh filename="file://$(find ros2srrc_endeffectors)/egp64/meshes/egp64_LeftFinger.dae" />
         </geometry>
+        <material name="black"/>
       </collision>
     </link>
@@ -158,8 +153,6 @@
       <inertial>
         <origin xyz="-0.0153 -0.00602 0" rpy="0 0 0" />
-        <mass value="0.02"/>
-        <inertia ixx="3.47e-07" ixy="0.0" ixz="0.0"
-                iyy="2.77e-06" iyz="0.0"
-                izz="2.91e-06"/>
+        <mass value="0.002" />
+        <inertia ixx="0.001" ixy="0.0" ixz="0.0" iyy="0.001" iyz="0.0" izz="0.001"/>
       </inertial>
       <visual>
@@ -173,4 +166,5 @@
           <mesh filename="file://$(find ros2srrc_endeffectors)/egp64/meshes/egp64_RightFingerBase.dae" />
         </geometry>
+        <material name="black"/>
       </collision>
     </link>
@@ -178,8 +172,8 @@
       <parent link="egp64_gripper_base_link" />
       <child link="egp64_finger_right_link" />
-      <limit effort="1000" lower="-0.0001" upper="0.027" velocity="0.2"/>
+      <limit effort="1000" lower="-0.001" upper="0.04" velocity="0.2"/>
       <origin xyz="-0.0153 -0.00602 0" rpy="0 0 0" />
       <axis xyz="1 0 0" />
-      <dynamics damping="0.2" friction="0.05"/>
+      <dynamics damping="1.0" friction="1.0"/>
     </joint>
     <!-- RIGHT FINGERTIP -->
@@ -187,8 +181,6 @@
       <inertial>
         <origin xyz="-0.01211 -0.00197 0.00093" rpy="0 0 0" />
-        <mass value="0.005"/>
-        <inertia ixx="3.71e-08" ixy="0.0" ixz="0.0"
-                iyy="1.77e-07" iyz="0.0"
-                izz="1.93e-07"/>
+        <mass value="0.001" />
+        <inertia ixx="0.001" ixy="0.0" ixz="0.0" iyy="0.001" iyz="0.0" izz="0.001"/>
       </inertial>
       <visual>
@@ -202,4 +194,5 @@
           <mesh filename="file://$(find ros2srrc_endeffectors)/egp64/meshes/egp64_RightFinger.dae" />
         </geometry>
+        <material name="black"/>
       </collision>
     </link>

File: src/abb_package/ros2_SimRealRobotControl/ros2srrc_endeffectors/egp64/urdf/egp64_ros2control.xacro (robot description, xacro)
@@ -33,6 +33,10 @@
     <joint name="egp64_finger_left_joint">
       <command_interface name="position">
-        <param name="min">-0.0001</param>
-        <param name="max">0.027</param>
+        <param name="min">-0.001</param>
+        <param name="max">0.04</param>
+      </command_interface>
+      <command_interface name="velocity">
+        <param name="min">-0.2</param>
+        <param name="max">0.2</param>
       </command_interface>
       <state_interface name="position">
@@ -44,6 +48,10 @@
     <joint name="egp64_finger_right_joint">
       <command_interface name="position">
-        <param name="min">-0.0001</param>
-        <param name="max">0.027</param>
+        <param name="min">-0.001</param>
+        <param name="max">0.04</param>
+      </command_interface>
+      <command_interface name="velocity">
+        <param name="min">-0.2</param>
+        <param name="max">0.2</param>
       </command_interface>
       <state_interface name="position">

File: src/abb_package/ros2_SimRealRobotControl/ros2srrc_endeffectors/egp64/urdf/egp64v2_macro.urdf.xacro (robot description, xacro)
@@ -76,6 +76,6 @@
           <mesh filename="file://$(find ros2srrc_endeffectors)/egp64/meshes/egp64_BaseNoAdapter.dae" />
         </geometry>
-        <material name="silver">
-          <color rgba="0.8 0.8 0.8 1"/>
+        <material name="blue">
+          <color rgba="0 0 1 1"/>
         </material>
       </visual>
@@ -84,4 +84,5 @@
           <mesh filename="file://$(find ros2srrc_endeffectors)/egp64/meshes/egp64_BaseNoAdapter.dae" />
         </geometry>
+        <material name="blue"/>
       </collision>
     </link>
@@ -116,8 +117,8 @@
       <parent link="egp64_gripper_base_link" />
       <child link="egp64_finger_left_link" />
-      <limit effort="1000" lower="-0.0001" upper="0.027" velocity="0.2"/>
+      <limit effort="1000" lower="-0.001" upper="0.04" velocity="0.2"/>
       <origin xyz="0.01483 -0.00782 0" rpy="0 0 0" />
       <axis xyz="-1 0 0" />
-      <dynamics damping="0.2" friction="0.05"/>
+      <dynamics damping="1.0" friction="1.0"/>
     </joint>
     <!-- LEFT FINGERTIP -->
@@ -171,8 +172,8 @@
       <parent link="egp64_gripper_base_link" />
       <child link="egp64_finger_right_link" />
-      <limit effort="1000" lower="-0.0001" upper="0.027" velocity="0.2"/>
+      <limit effort="1000" lower="-0.001" upper="0.04" velocity="0.2"/>
       <origin xyz="-0.0153 -0.00602 0" rpy="0 0 0" />
       <axis xyz="1 0 0" />
-      <dynamics damping="0.2" friction="0.05"/>
+      <dynamics damping="1.0" friction="1.0"/>
     </joint>
     <!-- RIGHT FINGERTIP -->

File: src/abb_package/ros2_SimRealRobotControl/ros2srrc_endeffectors/egp64/urdf/egp64v3_macro.urdf.xacro (robot description, xacro)
@@ -76,6 +76,6 @@
           <mesh filename="file://$(find ros2srrc_endeffectors)/egp64/meshes/egp64_BaseNoAdapter.dae" />
         </geometry>
-        <material name="silver">
-          <color rgba="0.8 0.8 0.8 1"/>
+        <material name="blue">
+          <color rgba="0 0 1 1"/>
         </material>
       </visual>
@@ -84,4 +84,5 @@
           <mesh filename="file://$(find ros2srrc_endeffectors)/egp64/meshes/egp64_BaseNoAdapter.dae" />
         </geometry>
+        <material name="blue"/>
       </collision>
     </link>
@@ -116,8 +117,8 @@
       <parent link="egp64_gripper_base_link" />
       <child link="egp64_finger_left_link" />
-      <limit effort="1000" lower="-0.0001" upper="0.027" velocity="0.2"/>
+      <limit effort="1000" lower="-0.001" upper="0.04" velocity="0.2"/>
       <origin xyz="0.01483 -0.00782 0" rpy="0 0 0" />
       <axis xyz="-1 0 0" />
-      <dynamics damping="0.2" friction="0.05"/>
+      <dynamics damping="1.0" friction="1.0"/>
     </joint>
     <!-- LEFT FINGERTIP -->
@@ -171,8 +172,8 @@
       <parent link="egp64_gripper_base_link" />
       <child link="egp64_finger_right_link" />
-      <limit effort="1000" lower="-0.0001" upper="0.027" velocity="0.2"/>
+      <limit effort="1000" lower="-0.001" upper="0.04" velocity="0.2"/>
       <origin xyz="-0.0153 -0.00602 0" rpy="0 0 0" />
       <axis xyz="1 0 0" />
-      <dynamics damping="0.2" friction="0.05"/>
+      <dynamics damping="1.0" friction="1.0"/>
     </joint>
     <!-- RIGHT FINGERTIP -->

File: src/abb_package/ros2_SimRealRobotControl/ros2srrc_endeffectors/gpp5010nc/urdf/gpp5010nc_macro.urdf.xacro (robot description, xacro)
@@ -48,7 +48,4 @@
           <mesh filename="file://$(find ros2srrc_endeffectors)/gpp5010nc/meshes/gpp5010nc_MainBody.dae" />
         </geometry>
-        <material name="silver">
-          <color rgba="0.8 0.8 0.8 1"/>
-        </material>
       </visual>
       <collision>
@@ -84,8 +81,8 @@
       <parent link="gpp5010nc_gripper_base_link" />
       <child link="gpp5010nc_finger_left_link" />
-      <limit effort="1000" lower="-0.0001" upper="0.0101" velocity="1.0"/>
+      <limit effort="1000" lower="-0.001" upper="0.011" velocity="1.0"/>
       <origin xyz="0.0 0.0 0.0" rpy="0 0 0" />
       <axis xyz="0 -1 0" />
-      <dynamics damping="0.2" friction="0.05"/>
+      <dynamics damping="1.0" friction="1.0"/>
     </joint>
     <!-- RIGHT FINGER -->
@@ -110,8 +107,8 @@
       <parent link="gpp5010nc_gripper_base_link" />
       <child link="gpp5010nc_finger_right_link" />
-      <limit effort="1000" lower="-0.0001" upper="0.0101" velocity="1.0"/>
+      <limit effort="1000" lower="-0.001" upper="0.011" velocity="1.0"/>
       <origin xyz="0.0 0.0 0.0" rpy="0 0 0" />
       <axis xyz="0 1 0" />
-      <dynamics damping="0.2" friction="0.05"/>
+      <dynamics damping="1.0" friction="1.0"/>
     </joint>
     <gazebo reference="gpp5010nc_finger_right_link">

File: src/abb_package/ros2_SimRealRobotControl/ros2srrc_endeffectors/gpp5010nc/urdf/gpp5010nc_ros2control.xacro (robot description, xacro)
@@ -33,6 +33,6 @@
     <joint name="gpp5010nc_finger_left_joint">
       <command_interface name="position">
-        <param name="min">-0.0001</param>
-        <param name="max">0.0101</param>
+        <param name="min">-0.001</param>
+        <param name="max">0.011</param>
       </command_interface>
       <command_interface name="velocity">
@@ -48,6 +48,6 @@
     <joint name="gpp5010nc_finger_right_joint">
       <command_interface name="position">
-        <param name="min">-0.0001</param>
-        <param name="max">0.0101</param>
+        <param name="min">-0.001</param>
+        <param name="max">0.011</param>
       </command_interface>
       <command_interface name="velocity">

File: src/abb_package/ros2_SimRealRobotControl/ros2srrc_endeffectors/ls_vgr/urdf/ls_vgr_macro.urdf.xacro (robot description, xacro)
@@ -48,7 +48,4 @@
           <mesh filename="file://$(find ros2srrc_endeffectors)/ls_vgr/meshes/ls_vgr.dae"/>
         </geometry>
-        <material name="silver">
-          <color rgba="0.8 0.8 0.8 1"/>
-        </material>
       </visual>
     </link>

File: src/abb_package/ros2_SimRealRobotControl/ros2srrc_endeffectors/robotiq_2f85/urdf/robotiq_2f85_macro.urdf.xacro (robot description, xacro)
@@ -116,6 +116,6 @@
       <axis xyz="0 0 1"/>
       <origin rpy="${pi} 0.0 0.0" xyz="0.05490451627 0.03060114443 0.0"/>
-      <limit lower="-0.0001" upper="0.8001" velocity="1.0" effort="1000"/>
-      <dynamics damping="0.2" friction="0.05"/>
+      <limit lower="-0.05" upper="0.80285" velocity="0.5" effort="1000"/>
+      <dynamics damping="1.0" friction="1.0"/>
     </joint>
     <!-- Robotiq: right_knuckle -->
@@ -139,11 +139,11 @@
       </inertial>
     </link>
-    <joint name="robotiq_85_right_knuckle_joint" type="revolute">
+    <joint name="robotiq_85_right_knuckle_joint" type="continuous">
       <parent link="robotiq_85_base_link"/>
       <child link="robotiq_85_right_knuckle_link"/>
       <axis xyz="0 0 1"/>
       <origin rpy="0.0 0.0 0.0" xyz="0.05490451627 -0.03060114443 0.0"/>
-      <limit lower="-0.0001" upper="0.8001" velocity="1.0" effort="1000"/>
-      <dynamics damping="0.2" friction="0.05"/>
+      <limit lower="-0.05" upper="0.80285" velocity="0.5" effort="1000"/>
+      <dynamics damping="1.0" friction="1.0"/>
     </joint>
     <!-- Robotiq: left_finger -->
@@ -171,4 +171,5 @@
       <child link="robotiq_85_left_finger_link"/>
       <origin xyz="-0.00408552455 -0.03148604435 0.0" rpy="0 0 0" />
+      <dynamics damping="1.0" friction="1.0"/>
     </joint>
     <!-- Robotiq: right_finger -->
@@ -196,4 +197,5 @@
       <child link="robotiq_85_right_finger_link"/>
       <origin xyz="-0.00408552455 -0.03148604435 0.0" rpy="0 0 0" />
+      <dynamics damping="1.0" friction="1.0"/>
     </joint>
     <!-- Robotiq: left_inner_knuckle -->
@@ -217,11 +219,11 @@
       </inertial>
     </link>
-    <joint name="robotiq_85_left_inner_knuckle_joint" type="revolute">
+    <joint name="robotiq_85_left_inner_knuckle_joint" type="continuous">
       <parent link="robotiq_85_base_link"/>
       <child link="robotiq_85_left_inner_knuckle_link"/>
       <axis xyz="0 0 1"/>
       <origin xyz="0.06142 0.0127 0" rpy="${pi} 0.0 0.0" />
-      <limit lower="-0.0001" upper="0.8001" velocity="1.0" effort="1000"/>
-      <dynamics damping="0.2" friction="0.05"/>
+      <limit lower="-0.05" upper="0.80285" velocity="0.5" effort="1000"/>
+      <dynamics damping="1.0" friction="1.0"/>
     </joint>
     <!-- Robotiq: right_inner_knuckle -->
@@ -245,11 +247,11 @@
       </inertial>
     </link>
-    <joint name="robotiq_85_right_inner_knuckle_joint" type="revolute">
+    <joint name="robotiq_85_right_inner_knuckle_joint" type="continuous">
       <parent link="robotiq_85_base_link"/>
       <child link="robotiq_85_right_inner_knuckle_link"/>
       <axis xyz="0 0 1"/>
       <origin xyz="0.06142 -0.0127 0" rpy="0 0 0"/>
-      <limit lower="-0.0001" upper="0.8001" velocity="1.0" effort="1000"/>
-      <dynamics damping="0.2" friction="0.05"/>
+      <limit lower="-0.05" upper="0.80285" velocity="0.5" effort="1000"/>
+      <dynamics damping="1.0" friction="1.0"/>
     </joint>
     <!-- Robotiq: left_finger_tip -->
@@ -273,11 +275,11 @@
       </inertial>
     </link>
-    <joint name="robotiq_85_left_finger_tip_joint" type="revolute">
+    <joint name="robotiq_85_left_finger_tip_joint" type="continuous">
       <parent link="robotiq_85_left_inner_knuckle_link"/>
       <child link="robotiq_85_left_finger_tip_link"/>
       <axis xyz="0 0 1"/>
       <origin xyz="0.04303959807 -0.03759940821 0.0" rpy="0.0 0.0 0.0"/>
-      <limit lower="-0.8001" upper="0.0001" velocity="1.0" effort="1000"/>
-      <dynamics damping="0.2" friction="0.05"/>
+      <limit lower="-0.80285" upper="0.05" velocity="0.5" effort="1000"/>
+      <dynamics damping="1.0" friction="1.0"/>
     </joint>
     <!-- Robotiq: right_finger_tip -->
@@ -301,11 +303,11 @@
       </inertial>
     </link>
-    <joint name="robotiq_85_right_finger_tip_joint" type="revolute">
+    <joint name="robotiq_85_right_finger_tip_joint" type="continuous">
       <parent link="robotiq_85_right_inner_knuckle_link"/>
       <child link="robotiq_85_right_finger_tip_link"/>
       <axis xyz="0 0 1"/>
       <origin rpy="0.0 0.0 0.0" xyz="0.04303959807 -0.03759940821  0.0"/>
-      <limit lower="-0.8001" upper="0.0001" velocity="1.0" effort="1000"/>
-      <dynamics damping="0.2" friction="0.05"/>
+      <limit lower="-0.80285" upper="0.05" velocity="0.5" effort="1000"/>
+      <dynamics damping="1.0" friction="1.0"/>
     </joint>
     <!-- SMALL CUBE FOR GRIPPER PLUGIN -->

File: src/abb_package/ros2_SimRealRobotControl/ros2srrc_endeffectors/robotiq_2f85/urdf/robotiq_2f85_ros2control.xacro (robot description, xacro)
@@ -32,6 +32,10 @@
     <joint name="robotiq_85_left_knuckle_joint">
       <command_interface name="position">
-        <param name="min">-0.0001</param>
-        <param name="max">0.8001</param>
+        <param name="min">-0.05</param>
+        <param name="max">0.80285</param>
+      </command_interface>
+      <command_interface name="velocity">
+        <param name="min">0.5</param>
+        <param name="max">0.5</param>
       </command_interface>
       <state_interface name="position">
@@ -43,6 +47,10 @@
     <joint name="robotiq_85_right_knuckle_joint">
       <command_interface name="position">
-        <param name="min">-0.0001</param>
-        <param name="max">0.8001</param>
+        <param name="min">-0.05</param>
+        <param name="max">0.80285</param>
+      </command_interface>
+      <command_interface name="velocity">
+        <param name="min">0.5</param>
+        <param name="max">0.5</param>
       </command_interface>
       <state_interface name="position">
@@ -54,6 +62,10 @@
     <joint name="robotiq_85_left_inner_knuckle_joint">
       <command_interface name="position">
-        <param name="min">-0.0001</param>
-        <param name="max">0.8001</param>
+        <param name="min">-0.05</param>
+        <param name="max">0.80285</param>
+      </command_interface>
+      <command_interface name="velocity">
+        <param name="min">0.5</param>
+        <param name="max">0.5</param>
       </command_interface>
       <state_interface name="position">
@@ -65,6 +77,10 @@
     <joint name="robotiq_85_right_inner_knuckle_joint">
       <command_interface name="position">
-        <param name="min">-0.0001</param>
-        <param name="max">0.8001</param>
+        <param name="min">-0.05</param>
+        <param name="max">0.80285</param>
+      </command_interface>
+      <command_interface name="velocity">
+        <param name="min">0.5</param>
+        <param name="max">0.5</param>
       </command_interface>
       <state_interface name="position">
@@ -76,6 +92,10 @@
     <joint name="robotiq_85_left_finger_tip_joint">
       <command_interface name="position">
-        <param name="min">-0.8001</param>
-        <param name="max">0.0001</param>
+        <param name="min">-0.80285</param>
+        <param name="max">0.05</param>
+      </command_interface>
+      <command_interface name="velocity">
+        <param name="min">0.5</param>
+        <param name="max">0.5</param>
       </command_interface>
       <state_interface name="position">
@@ -87,6 +107,10 @@
     <joint name="robotiq_85_right_finger_tip_joint">
       <command_interface name="position">
-        <param name="min">-0.8001</param>
-        <param name="max">0.0001</param>
+        <param name="min">-0.80285</param>
+        <param name="max">0.05</param>
+      </command_interface>
+      <command_interface name="velocity">
+        <param name="min">0.5</param>
+        <param name="max">0.5</param>
       </command_interface>
       <state_interface name="position">
