Commit message: controllers shaghala inshallah

File: src/abb_package/ros2_SimRealRobotControl/ros2srrc_endeffectors/robotiq_hande/urdf/robotiq_hande_macro.urdf.xacro (robot description, xacro)
@@ -37,5 +37,5 @@
     </xacro:unless>
     <!-- ***** Robotiq HandE GRIPPER .urdf SERIAL CHAIN ***** -->
-    <!-- Robotiq: bracket
+    <!-- Robotiq: bracket -->
     <link name="robotiq_bracket">
       <visual>
@@ -60,5 +60,5 @@
       <parent link="${parent_link}"/>
       <child link="robotiq_bracket"/>
-    </joint> -->
+    </joint>
     <!-- Robotiq: coupler -->
     <link name="robotiq_coupler">
@@ -67,7 +67,4 @@
           <mesh filename="file://$(find ros2srrc_endeffectors)/robotiq_hande/meshes/robotiq_hande_coupler.stl" />
         </geometry>
-        <material name="dark_grey">
-          <color rgba="0.2 0.2 0.2 1"/>
-        </material>
       </visual>
       <collision>
@@ -84,6 +81,6 @@
     </link>
     <joint name="robotiq_coupler_joint" type="fixed">
-      <origin xyz="0 0 -0.008" rpy="0 0 0" />
-      <parent link="${parent_link}"/>
+      <origin xyz="0 0 0" rpy="0 0 0" />
+      <parent link="robotiq_bracket"/>
       <child link="robotiq_coupler"/>
     </joint>
@@ -124,5 +121,5 @@
         <origin rpy="0 0 0" xyz="0.02262 -0.00759 0.00738"/>
         <mass value="0.03804"/>
-        <inertia ixx="1.3567e-05" ixy="0" ixz="0" iyy="1.5784e-05" iyz="0" izz="7.478e-06"/>
+        <inertia ixx="13567E-9" ixy="1849E-9" ixz="3622E-9" iyy="15784E-9" iyz="3616E-9" izz="7478E-9"/>
       </inertial>
       <visual>
@@ -131,7 +128,4 @@
           <mesh filename="file://$(find ros2srrc_endeffectors)/robotiq_hande/meshes/finger_1.dae"/>
         </geometry>
-        <material name="dark_grey">
-          <color rgba="0.2 0.2 0.2 1"/>
-        </material>
       </visual>
       <collision>
@@ -142,4 +136,7 @@
       </collision>
     </link>
+    <gazebo reference="robotiq_hande_left_finger">
+      <material>Gazebo/Grey</material>
+    </gazebo>
     <joint name="robotiq_hande_left_finger_joint" type="prismatic">
       <origin rpy="0 0 0" xyz="0.0 0.0 0.099"/>
@@ -147,6 +144,5 @@
       <child link="robotiq_hande_left_finger"/>
       <axis xyz="-1 0 0"/>
-      <limit effort="130" lower="-0.0001" upper="0.0251" velocity="0.15"/>
-      <dynamics damping="0.2" friction="0.05"/>
+      <limit effort="130" lower="-0.05" upper="0.025" velocity="0.15"/>
     </joint>
     <!-- Robotiq: right finger -->
@@ -155,5 +151,5 @@
         <origin rpy="0 0 0" xyz="-0.02262 0.00759 0.00738"/>
         <mass value="0.03804"/>
-        <inertia ixx="1.3567e-05" ixy="0" ixz="0" iyy="1.5784e-05" iyz="0" izz="7.478e-06"/>
+        <inertia ixx="13567E-9" ixy="1849E-9" ixz="3622E-9" iyy="15784E-9" iyz="3616E-9" izz="7478E-9"/>
       </inertial>
       <visual>
@@ -162,7 +158,4 @@
           <mesh filename="file://$(find ros2srrc_endeffectors)/robotiq_hande/meshes/finger_2.dae"/>
         </geometry>
-        <material name="dark_grey">
-          <color rgba="0.2 0.2 0.2 1"/>
-        </material>
       </visual>
       <collision>
@@ -173,4 +166,7 @@
       </collision>
     </link>
+    <gazebo reference="robotiq_hande_right_finger">
+      <material>Gazebo/Grey</material>
+    </gazebo>
     <joint name="robotiq_hande_right_finger_joint" type="prismatic">
       <origin rpy="0 0 0" xyz="0 0 0.099"/>
@@ -178,6 +174,5 @@
       <child link="robotiq_hande_right_finger"/>
       <axis xyz="1 0 0"/>
-      <limit effort="130" lower="-0.0001" upper="0.0251" velocity="0.15"/>
-      <dynamics damping="0.2" friction="0.05"/>
+      <limit effort="130" lower="-0.05" upper="0.025" velocity="0.15"/>
     </joint>
     <!-- SMALL CUBE FOR GRIPPER PLUGIN -->

File: src/abb_package/ros2_SimRealRobotControl/ros2srrc_endeffectors/robotiq_hande/urdf/robotiq_hande_ros2control.xacro (robot description, xacro)
@@ -32,6 +32,6 @@
     <joint name="robotiq_hande_left_finger_joint">
       <command_interface name="position">
-        <param name="min">-0.0001</param>
-        <param name="max">0.0251</param>
+        <param name="min">-0.05</param>
+        <param name="max">0.025</param>
       </command_interface>
       <command_interface name="velocity">
@@ -47,6 +47,6 @@
     <joint name="robotiq_hande_right_finger_joint">
       <command_interface name="position">
-        <param name="min">-0.0001</param>
-        <param name="max">0.0251</param>
+        <param name="min">-0.05</param>
+        <param name="max">0.025</param>
       </command_interface>
       <command_interface name="velocity">

File: src/abb_package/ros2_SimRealRobotControl/ros2srrc_endeffectors/robotiq_hande/urdf/robotiq_handev2_macro.urdf.xacro (robot description, xacro)
@@ -37,5 +37,5 @@
     </xacro:unless>
     <!-- ***** Robotiq HandE GRIPPER .urdf SERIAL CHAIN ***** -->
-    <!-- Robotiq: bracket
+    <!-- Robotiq: bracket -->
     <link name="robotiq_bracket">
       <visual>
@@ -60,5 +60,5 @@
       <parent link="${parent_link}"/>
       <child link="robotiq_bracket"/>
-    </joint> -->
+    </joint>
     <!-- Robotiq: coupler -->
     <link name="robotiq_coupler">
@@ -67,7 +67,4 @@
           <mesh filename="file://$(find ros2srrc_endeffectors)/robotiq_hande/meshes/robotiq_hande_coupler.stl" />
         </geometry>
-        <material name="dark_grey">
-          <color rgba="0.2 0.2 0.2 1"/>
-        </material>
       </visual>
       <collision>
@@ -84,8 +81,13 @@
     </link>
     <joint name="robotiq_coupler_joint" type="fixed">
-      <origin xyz="0 0 -0.008" rpy="0 0 0" />
-      <parent link="${parent_link}"/>
+      <origin xyz="0 0 0" rpy="0 0 0" />
+      <parent link="robotiq_bracket"/>
       <child link="robotiq_coupler"/>
     </joint>
+    <gazebo reference="robotiq_coupler">
+      <mu1>0.9</mu1>
+      <mu2>0.9</mu2>
+      <material>Gazebo/FlatBlack</material>
+    </gazebo>
     <!-- Robotiq: base_link -->
     <link name="robotiq_hande_base_link">
@@ -119,5 +121,5 @@
         <origin rpy="0 0 0" xyz="0.02262 -0.00759 0.00738"/>
         <mass value="0.03804"/>
-        <inertia ixx="1.3567e-05" ixy="0" ixz="0" iyy="1.5784e-05" iyz="0" izz="7.478e-06"/>
+        <inertia ixx="13567E-9" ixy="1849E-9" ixz="3622E-9" iyy="15784E-9" iyz="3616E-9" izz="7478E-9"/>
       </inertial>
       <visual>
@@ -126,7 +128,4 @@
           <mesh filename="file://$(find ros2srrc_endeffectors)/robotiq_hande/meshes/finger_1v2.dae"/>
         </geometry>
-        <material name="dark_grey">
-          <color rgba="0.2 0.2 0.2 1"/>
-        </material>
       </visual>
       <collision>
@@ -137,4 +136,7 @@
       </collision>
     </link>
+    <gazebo reference="robotiq_hande_left_finger">
+      <material>Gazebo/Grey</material>
+    </gazebo>
     <joint name="robotiq_hande_left_finger_joint" type="prismatic">
       <origin rpy="0 0 0" xyz="0.0 0.0 0.099"/>
@@ -142,6 +144,5 @@
       <child link="robotiq_hande_left_finger"/>
       <axis xyz="-1 0 0"/>
-      <limit effort="130" lower="-0.0001" upper="0.0251" velocity="0.15"/>
-      <dynamics damping="0.2" friction="0.05"/>
+      <limit effort="130" lower="-0.05" upper="0.025" velocity="0.15"/>
     </joint>
     <!-- Robotiq: right finger -->
@@ -150,5 +151,5 @@
         <origin rpy="0 0 0" xyz="-0.02262 0.00759 0.00738"/>
         <mass value="0.03804"/>
-        <inertia ixx="1.3567e-05" ixy="0" ixz="0" iyy="1.5784e-05" iyz="0" izz="7.478e-06"/>
+        <inertia ixx="13567E-9" ixy="1849E-9" ixz="3622E-9" iyy="15784E-9" iyz="3616E-9" izz="7478E-9"/>
       </inertial>
       <visual>
@@ -157,7 +158,4 @@
           <mesh filename="file://$(find ros2srrc_endeffectors)/robotiq_hande/meshes/finger_2v2.dae"/>
         </geometry>
-        <material name="dark_grey">
-          <color rgba="0.2 0.2 0.2 1"/>
-        </material>
       </visual>
       <collision>
@@ -168,4 +166,7 @@
       </collision>
     </link>
+    <gazebo reference="robotiq_hande_right_finger">
+      <material>Gazebo/Grey</material>
+    </gazebo>
     <joint name="robotiq_hande_right_finger_joint" type="prismatic">
       <origin rpy="0 0 0" xyz="0 0 0.099"/>
@@ -173,6 +174,5 @@
       <child link="robotiq_hande_right_finger"/>
       <axis xyz="1 0 0"/>
-      <limit effort="130" lower="-0.0001" upper="0.0251" velocity="0.15"/>
-      <dynamics damping="0.2" friction="0.05"/>
+      <limit effort="130" lower="-0.05" upper="0.025" velocity="0.15"/>
     </joint>
     <!-- SMALL CUBE FOR GRIPPER PLUGIN -->

File: src/abb_package/ros2_SimRealRobotControl/ros2srrc_robots/irb120/urdf/irb120_macro.urdf.xacro (robot description, xacro)
@@ -37,5 +37,5 @@
 #  COPYRIGHT - ROS-Industrial                                                           #
 #  (ORIGINAL LICENSE) -> Licensed under the Apache-2.0 License.                         #
-#                                                                                       #
+#                     abb_table                                                                  #
 #  CHANGES MADE:                                                                        #
 #  The original files contain the .urdf information of the robot for ROS1, and these    #
@@ -58,5 +58,5 @@
     </xacro:unless>
     <!-- ABB-IRB120 GAZEBO - ROS2_CONTROL: -->
-    <xacro:include filename="$(find ros2srrc_robots)/irb120/urdf/irb120_ros2control.xacro" />
+    <!--<xacro:include filename="$(find ros2srrc_robots)/irb120/urdf/irb120_ros2control.xacro" />
     <xacro:irb120_ros2control
       bringup="${bringup}"
@@ -64,5 +64,5 @@
       EE="${EE}"
       EE_name="${EE_name}"
-    />
+    /> -->
     <!-- ***** ABB-IRB120 ROBOT .urdf SERIAL CHAIN ***** -->
     <!-- Link list: -->
@@ -79,4 +79,5 @@
           <mesh filename="file://$(find ros2srrc_robots)/irb120/meshes/visual/base_link.dae"/>
         </geometry>
+        <xacro:material_abb_orange />
       </visual>
       <collision>
@@ -100,4 +101,5 @@
           <mesh filename="file://$(find ros2srrc_robots)/irb120/meshes/visual/link_1.dae"/>
         </geometry>
+        <xacro:material_abb_orange />
       </visual>
       <collision>
@@ -121,4 +123,5 @@
           <mesh filename="file://$(find ros2srrc_robots)/irb120/meshes/visual/link_2.dae"/>
         </geometry>
+        <xacro:material_abb_orange />
       </visual>
       <collision>
@@ -142,4 +145,5 @@
           <mesh filename="file://$(find ros2srrc_robots)/irb120/meshes/visual/link_3.dae"/>
         </geometry>
+        <xacro:material_abb_orange />
       </visual>
       <collision>
@@ -163,4 +167,5 @@
           <mesh filename="file://$(find ros2srrc_robots)/irb120/meshes/visual/link_4.dae"/>
         </geometry>
+        <xacro:material_abb_orange />
       </visual>
       <collision>
@@ -184,4 +189,5 @@
           <mesh filename="file://$(find ros2srrc_robots)/irb120/meshes/visual/link_5.dae"/>
         </geometry>
+        <xacro:material_abb_orange />
       </visual>
       <collision>
@@ -205,4 +211,5 @@
           <mesh filename="file://$(find ros2srrc_robots)/irb120/meshes/visual/link_6.dae"/>
         </geometry>
+        <xacro:material_abb_black />
       </visual>
       <collision>
@@ -223,5 +230,5 @@
       <limit effort="1000" lower="-2.87979" upper="2.87979" velocity="4.36332"/>
       <axis xyz="0 0 1"/>
-      <dynamics damping="1.0" friction="0.0"/>
+      <dynamics damping="50.0" friction="1.0"/>
     </joint>
     <!-- joint_2 -->
@@ -232,5 +239,5 @@
       <limit effort="1000" lower="-1.91986" upper="1.91986" velocity="4.36332"/>
       <axis xyz="0 1 0"/>
-      <dynamics damping="0.5" friction="0.0"/>
+      <dynamics damping="50.0" friction="1.0"/>
     </joint>
     <!-- joint_3 -->
@@ -241,5 +248,5 @@
       <limit effort="1000" lower="-1.91986" upper="1.22173" velocity="4.36332"/>
       <axis xyz="0 1 0"/>
-      <dynamics damping="0.3" friction="0.0"/>
+      <dynamics damping="10.0" friction="1.0"/>
     </joint>
     <!-- joint_4 -->
@@ -250,5 +257,5 @@
       <limit effort="1000" lower="-2.79253" upper="2.79253" velocity="5.58505"/>
       <axis xyz="1 0 0"/>
-      <dynamics damping="0.1" friction="0.0"/>
+      <dynamics damping="5.0" friction="1.0"/>
     </joint>
     <!-- joint_5 -->
@@ -259,5 +266,5 @@
       <limit effort="1000" lower="-2.094395" upper="2.094395" velocity="5.58505"/>
       <axis xyz="0 1 0"/>
-      <dynamics damping="0.05" friction="0.0"/>
+      <dynamics damping="2.0" friction="1.0"/>
     </joint>
     <!-- joint_6 -->
@@ -268,5 +275,5 @@
       <limit effort="1000" lower="-6.98132" upper="6.98132" velocity="7.33038"/>
       <axis xyz="1 0 0"/>
-      <dynamics damping="0.01" friction="0.0"/>
+      <dynamics damping="1.0" friction="1.0"/>
     </joint>
     <!-- end of joint list -->

File: src/abb_package/ros2_SimRealRobotControl/ros2srrc_robots/irb120/urdf/irb120_ros2control.xacro (robot description, xacro)
@@ -138,5 +138,5 @@
       <joint name="joint_5">
         <command_interface name="position">
-          <param name="min">-2.00</param>       <!-- Joint5 limits lowered to +-2rad -->
+          <param name="min">-2.00</param>
           <param name="max">2.00</param>
         </command_interface>
