Commit message: fixed controllers and solver problems Integrated the GUI into the supervisor

File: src/abb_package/ros2_SimRealRobotControl/ros2srrc_robots/irb120/urdf/irb120_macro.urdf.xacro (robot description, xacro)
@@ -37,5 +37,5 @@
 #  COPYRIGHT - ROS-Industrial                                                           #
 #  (ORIGINAL LICENSE) -> Licensed under the Apache-2.0 License.                         #
-#                                                                                       #
+#                     abb_table                                                                  #
 #  CHANGES MADE:                                                                        #
 #  The original files contain the .urdf information of the robot for ROS1, and these    #
@@ -58,5 +58,5 @@
     </xacro:unless>
     <!-- ABB-IRB120 GAZEBO - ROS2_CONTROL: -->
-    <xacro:include filename="$(find ros2srrc_robots)/irb120/urdf/irb120_ros2control.xacro" />
+    <!-- <xacro:include filename="$(find ros2srrc_robots)/irb120/urdf/irb120_ros2control.xacro" />
     <xacro:irb120_ros2control
       bringup="${bringup}"
@@ -64,5 +64,5 @@
       EE="${EE}"
       EE_name="${EE_name}"
-    />
+    /> -->
     <!-- ***** ABB-IRB120 ROBOT .urdf SERIAL CHAIN ***** -->
     <!-- Link list: -->
@@ -79,4 +79,5 @@
           <mesh filename="file://$(find ros2srrc_robots)/irb120/meshes/visual/base_link.dae"/>
         </geometry>
+        <xacro:material_abb_orange />
       </visual>
       <collision>
@@ -100,4 +101,5 @@
           <mesh filename="file://$(find ros2srrc_robots)/irb120/meshes/visual/link_1.dae"/>
         </geometry>
+        <xacro:material_abb_orange />
       </visual>
       <collision>
@@ -121,4 +123,5 @@
           <mesh filename="file://$(find ros2srrc_robots)/irb120/meshes/visual/link_2.dae"/>
         </geometry>
+        <xacro:material_abb_orange />
       </visual>
       <collision>
@@ -142,4 +145,5 @@
           <mesh filename="file://$(find ros2srrc_robots)/irb120/meshes/visual/link_3.dae"/>
         </geometry>
+        <xacro:material_abb_orange />
       </visual>
       <collision>
@@ -163,4 +167,5 @@
           <mesh filename="file://$(find ros2srrc_robots)/irb120/meshes/visual/link_4.dae"/>
         </geometry>
+        <xacro:material_abb_orange />
       </visual>
       <collision>
@@ -184,4 +189,5 @@
           <mesh filename="file://$(find ros2srrc_robots)/irb120/meshes/visual/link_5.dae"/>
         </geometry>
+        <xacro:material_abb_orange />
       </visual>
       <collision>
@@ -205,4 +211,5 @@
           <mesh filename="file://$(find ros2srrc_robots)/irb120/meshes/visual/link_6.dae"/>
         </geometry>
+        <xacro:material_abb_black />
       </visual>
       <collision>
@@ -223,5 +230,5 @@
       <limit effort="1000" lower="-2.87979" upper="2.87979" velocity="4.36332"/>
       <axis xyz="0 0 1"/>
-      <dynamics damping="1.0" friction="0.0"/>
+      <dynamics damping="50.0" friction="1.0"/>
     </joint>
     <!-- joint_2 -->
@@ -232,5 +239,5 @@
       <limit effort="1000" lower="-1.91986" upper="1.91986" velocity="4.36332"/>
       <axis xyz="0 1 0"/>
-      <dynamics damping="0.5" friction="0.0"/>
+      <dynamics damping="50.0" friction="1.0"/>
     </joint>
     <!-- joint_3 -->
@@ -241,5 +248,5 @@
       <limit effort="1000" lower="-1.91986" upper="1.22173" velocity="4.36332"/>
       <axis xyz="0 1 0"/>
-      <dynamics damping="0.3" friction="0.0"/>
+      <dynamics damping="10.0" friction="1.0"/>
     </joint>
     <!-- joint_4 -->
@@ -250,5 +257,5 @@
       <limit effort="1000" lower="-2.79253" upper="2.79253" velocity="5.58505"/>
       <axis xyz="1 0 0"/>
-      <dynamics damping="0.1" friction="0.0"/>
+      <dynamics damping="5.0" friction="1.0"/>
     </joint>
     <!-- joint_5 -->
@@ -259,5 +266,5 @@
       <limit effort="1000" lower="-2.094395" upper="2.094395" velocity="5.58505"/>
       <axis xyz="0 1 0"/>
-      <dynamics damping="0.05" friction="0.0"/>
+      <dynamics damping="2.0" friction="1.0"/>
     </joint>
     <!-- joint_6 -->
@@ -268,5 +275,5 @@
       <limit effort="1000" lower="-6.98132" upper="6.98132" velocity="7.33038"/>
       <axis xyz="1 0 0"/>
-      <dynamics damping="0.01" friction="0.0"/>
+      <dynamics damping="1.0" friction="1.0"/>
     </joint>
     <!-- end of joint list -->

File: src/dual_arms/urdf/dual_arms_with_environment.xacro (robot description, xacro)
@@ -1,4 +1,5 @@
 <?xml version="1.0" ?>
 <robot name="dual_arms_with_environment" xmlns:xacro="http://www.ros.org/wiki/xacro">
+  <xacro:arg name="bringup" default="false"/>
   <xacro:include filename="$(find assembly_environment)/urdf/environment.xacro" />
   <xacro:include filename="$(find annin_ar4_description)/urdf/ar_macro.xacro" />
@@ -37,61 +38,45 @@
   </xacro:irb120_mounted>
   <xacro:abb_gripper arm_parent_link="tool0" gripper_prefix="gripper_"/>
- <!-- <link name="Base_brick">
-    <visual>
-      <origin xyz="0 0 0" rpy="0 0 0"/>
-      <geometry>
-        <mesh filename="file:///home/mohamed/full_system/src/dual_arms/meshes/bricks/base_brick.STL" scale="0.001 0.001 0.001"/>
-      </geometry>
-      <material name="Black">
-        <color rgba="0.0 0.0 0.0 1.0"/>
-      </material>
-    </visual>
-    <collision>
-      <origin xyz="0 0 0" rpy="0 0 0"/>
-      <geometry>
-        <mesh filename="file:///home/mohamed/full_system/src/dual_arms/meshes/bricks/base_brick.STL" scale="0.001 0.001 0.001"/>
-      </geometry>
-    </collision>
-    <inertial>
-      <mass value="1.0"/>
-      <inertia ixx="0.1" ixy="0.0" ixz="0.0" iyy="0.1" iyz="0.0" izz="0.1"/>
-    </inertial>
-  </link>
-  <gazebo reference="Base_brick">
-    <material>Gazebo/Black</material>
+  <gazebo reference="ar4_gripper_jaw1_link">
+    <mu1>100.0</mu1>
+    <mu2>100.0</mu2>
+    <minDepth>0.001</minDepth>
+    <maxVel>0.0</maxVel>
   </gazebo>
-    <joint name="world_to_base_brick_joint" type="fixed">
-    <parent link="world"/>
-    <child link="Base_brick"/>
-    <origin xyz="0.6 0 1.1" rpy="0 0 0"/>
-  </joint>
-    <link name="T_brick_1">
-    <visual>
-      <origin xyz="0 0 0" rpy="0 0 0"/>
-      <geometry>
-        <mesh filename="file:///home/mohamed/full_system/src/dual_arms/meshes/bricks/T_brick.STL" scale="0.001 0.001 0.001"/>
-      </geometry>
-      <material name="Blue">
-        <color rgba="0.0 0.0 1.0 1.0"/>
-      </material>
-    </visual>
-    <collision>
-      <origin xyz="0 0 0" rpy="0 0 0"/>
-      <geometry>
-        <mesh filename="file:///home/mohamed/full_system/src/dual_arms/meshes/bricks/T_brick.STL" scale="0.001 0.001 0.001"/>
-      </geometry>
-    </collision>
-    <inertial>
-      <mass value="1.0"/>
-      <inertia ixx="0.1" ixy="0.0" ixz="0.0" iyy="0.1" iyz="0.0" izz="0.1"/>
-    </inertial>
-  </link>
-  <gazebo reference="T_brick_1">
-    <material>Gazebo/Blue</material>
+  <gazebo reference="ar4_gripper_jaw2_link">
+    <mu1>100.0</mu1>
+    <mu2>100.0</mu2>
+    <minDepth>0.001</minDepth>
+    <maxVel>0.0</maxVel>
   </gazebo>
-  <joint name="world_to_T_brick_1" type="fixed">
-    <parent link="world"/>
-    <child link="T_brick_1"/>
-    <origin xyz="0.6 0 1.14" rpy="0 0 0"/>
-  </joint> -->
+  <gazebo reference="gripper_ABB_Gripper_Finger_1">
+    <mu1>100.0</mu1>
+    <mu2>100.0</mu2>
+    <minDepth>0.001</minDepth>
+    <maxVel>0.0</maxVel>
+  </gazebo>
+  <gazebo reference="gripper_ABB_Gripper_Finger_2">
+    <mu1>100.0</mu1>
+    <mu2>100.0</mu2>
+    <minDepth>0.001</minDepth>
+    <maxVel>0.0</maxVel>
+  </gazebo>
+  <gazebo>
+    <plugin filename="libgz-sim-vacuum-gripper-system.so"
+            name="gz::sim::systems::VacuumGripper">
+        <link_name>ar4_gripper_jaw1_link</link_name>
+        <suction_enabled>false</suction_enabled>
+        <fixed>false</fixed>
+        <suction_on_topic>/ar4/gripper/lock_trigger</suction_on_topic>
+        <contact_sensor_topic>/ar4/gripper/contact</contact_sensor_topic>
+    </plugin>
+    <plugin filename="libgz-sim-vacuum-gripper-system.so"
+            name="gz::sim::systems::VacuumGripper">
+        <link_name>gripper_ABB_Gripper_Finger_1</link_name>
+        <suction_enabled>false</suction_enabled>
+        <fixed>false</fixed>
+        <suction_on_topic>/abb/gripper/lock_trigger</suction_on_topic>
+        <contact_sensor_topic>/abb/gripper/contact</contact_sensor_topic>
+    </plugin>
+  </gazebo>
 </robot>
