Commit message: added ABB_base_link for testing pose commands given in reference to ABB base frame

File: src/ar4_package/annin_ar4_description/urdf/ar_gazebo.urdf.xacro (robot description, xacro)
@@ -9,35 +9,20 @@
   <xacro:arg name="include_gripper" default="True" />
   <link name="world" />
-  <xacro:ar_robot
-    tf_prefix="$(arg tf_prefix)"
-    parent="world"
-    robot_parameters_file="$(find annin_ar4_description)/config/$(arg ar_model).yaml"
-  >
+  <link name="ABB_base_link" />
+  <joint name="ABB_base_link_to_world_joint" type="fixed">
+    <parent link="world" />
+    <child link="ABB_base_link" />
+    <origin xyz="0 -1.110
+      0" rpy="0 0 0" />
+  </joint>
+  <xacro:ar_robot tf_prefix="$(arg tf_prefix)" parent="world" robot_parameters_file="$(find annin_ar4_description)/config/$(arg ar_model).yaml">
     <origin xyz="0 0 0" rpy="0 0 0" />
   </xacro:ar_robot>
   <xacro:if value="$(arg include_gripper)">
     <xacro:include filename="$(find annin_ar4_description)/urdf/ar_gripper_macro.xacro" />
-    <xacro:ar_gripper
-      tf_prefix="$(arg tf_prefix)"
-      parent="$(arg tf_prefix)ee_link"
-    />
-    <xacro:ar_gripper_ros2_control
-      name="ARGripperGazeboSystem"
-      plugin_name="gz_ros2_control/GazeboSimSystem"
-      serial_port="None"
-      driver_parameters_file="$(find annin_ar4_driver)/config/gripper_driver.yaml"
-      tf_prefix="$(arg tf_prefix)"
-    />
+    <xacro:ar_gripper tf_prefix="$(arg tf_prefix)" parent="$(arg tf_prefix)ee_link" />
+    <xacro:ar_gripper_ros2_control name="ARGripperGazeboSystem" plugin_name="gz_ros2_control/GazeboSimSystem" serial_port="None" driver_parameters_file="$(find annin_ar4_driver)/config/gripper_driver.yaml" tf_prefix="$(arg tf_prefix)" />
   </xacro:if>
-  <xacro:ar_ros2_control
-    ar_model="$(arg ar_model)"
-    plugin_name="gz_ros2_control/GazeboSimSystem"
-    serial_port="None"
-    calibrate="False"
-    robot_parameters_file="$(find annin_ar4_description)/config/$(arg ar_model).yaml"
-    joint_offset_parameters_file="$(find annin_ar4_driver)/config/joint_offsets/$(arg ar_model).yaml"
-    driver_parameters_file="$(find annin_ar4_driver)/config/driver.yaml"
-    tf_prefix="$(arg tf_prefix)"
-  />
+  <xacro:ar_ros2_control ar_model="$(arg ar_model)" plugin_name="gz_ros2_control/GazeboSimSystem" serial_port="None" calibrate="False" robot_parameters_file="$(find annin_ar4_description)/config/$(arg ar_model).yaml" joint_offset_parameters_file="$(find annin_ar4_driver)/config/joint_offsets/$(arg ar_model).yaml" driver_parameters_file="$(find annin_ar4_driver)/config/driver.yaml" tf_prefix="$(arg tf_prefix)" />
   <gazebo reference="world" />
   <gazebo>
