Commit message: modified ar4 files: removed abb dummy link and edited pose commander

File: src/ar4_package/annin_ar4_description/urdf/ar.urdf.xacro (robot description, xacro)
@@ -6,11 +6,4 @@
   <xacro:include filename="$(find annin_ar4_description)/urdf/ar_gripper_macro.xacro" />
   <link name="world" />
-  <link name="Abb_dummy_base" />
-  <joint name="ABB_base_joint" type="fixed">
-    <parent link="world" />
-    <child link="Abb_dummy_base" />
-    <origin xyz="0 -1.110
-      0" rpy="0 0 0" />
-  </joint>
   <xacro:ar_robot
     tf_prefix="$(arg tf_prefix)"

File: src/ar4_package/annin_ar4_description/urdf/ar_gazebo.urdf.xacro (robot description, xacro)
@@ -9,10 +9,4 @@
   <xacro:arg name="include_gripper" default="True" />
   <link name="world" />
-  <link name="Abb_dummy_base" />
-  <joint name="ABB_base_joint" type="fixed">
-    <parent link="world" />
-    <child link="Abb_dummy_base" />
-    <origin xyz="0 -1.110  0" rpy="0 0 0" />
-  </joint>
   <xacro:ar_robot
     tf_prefix="$(arg tf_prefix)"

File: src/dual_arms/urdf/dual_arms_with_environment.xacro (robot description, xacro)
@@ -62,6 +62,6 @@
     <maxVel>0.0</maxVel>
   </gazebo>
-  <gazebo>
-    <plugin filename="libgz-sim-vacuum-gripper-system.so"
+   <gazebo>
+    <plugin filename="gz-sim-vacuum-gripper-system"
             name="gz::sim::systems::VacuumGripper">
         <link_name>ar4_gripper_jaw1_link</link_name>
@@ -71,5 +71,5 @@
         <contact_sensor_topic>/ar4/gripper/contact</contact_sensor_topic>
     </plugin>
-    <plugin filename="libgz-sim-vacuum-gripper-system.so"
+    <plugin filename="gz-sim-vacuum-gripper-system"
             name="gz::sim::systems::VacuumGripper">
         <link_name>gripper_ABB_Gripper_Finger_1</link_name>

Commit message: added ABB_base_Link for testing pose commands given in reference to ABB base frame

File: src/ar4_package/annin_ar4_description/urdf/ar.urdf.xacro (robot description, xacro)
@@ -6,16 +6,16 @@
   <xacro:include filename="$(find annin_ar4_description)/urdf/ar_gripper_macro.xacro" />
   <link name="world" />
-  <xacro:ar_robot
-    tf_prefix="$(arg tf_prefix)"
-    parent="world"
-    robot_parameters_file="$(find annin_ar4_description)/config/$(arg ar_model).yaml"
-  >
+  <link name="ABB_base_link" />
+  <joint name="ABB_base_link_to_world_joint" type="fixed">
+    <parent link="world" />
+    <child link="ABB_base_link" />
+    <origin xyz="0 -1.110
+      0" rpy="0 0 0" />
+  </joint>
+  <xacro:ar_robot tf_prefix="$(arg tf_prefix)" parent="world" robot_parameters_file="$(find annin_ar4_description)/config/$(arg ar_model).yaml">
     <origin xyz="0 0 0" rpy="0 0 0" />
   </xacro:ar_robot>
   <xacro:if value="$(arg include_gripper)">
-    <xacro:ar_gripper
-      tf_prefix="$(arg tf_prefix)"
-      parent="$(arg tf_prefix)ee_link"
-    />
+    <xacro:ar_gripper tf_prefix="$(arg tf_prefix)" parent="$(arg tf_prefix)ee_link" />
   </xacro:if>
 </robot>
