Commit message: fix: ar4 gripper control

File: src/ar4_package/annin_ar4_description/urdf/ar_gripper.ros2_control.xacro (robot description, xacro)
@@ -28,5 +28,5 @@
         </state_interface>
       </joint>
-      <joint name="${tf_prefix}gripper_jaw2_joint">
+      <!-- <joint name="${tf_prefix}gripper_jaw2_joint">
         <param name="mimic">${tf_prefix}gripper_jaw1_joint</param>
         <param name="multiplier">1</param>
@@ -37,5 +37,5 @@
           <param name="initial_value">0.0</param>
         </state_interface>
-      </joint>
+      </joint> -->
     </ros2_control>
   </xacro:macro>

File: src/dual_arms/urdf/dual_arms.gazebo.xacro (robot description, xacro)
@@ -23,5 +23,5 @@
     <joint name="joint_6"><command_interface name="position"/><state_interface name="position"/><state_interface name="velocity"/></joint>
     <joint name="ar4_gripper_jaw1_joint"><command_interface name="position"/><state_interface name="position"/><state_interface name="velocity"/></joint>
-    <joint name="ar4_gripper_jaw2_joint"><command_interface name="position"/><state_interface name="position"/><state_interface name="velocity"/></joint>
+    <!-- <joint name="ar4_gripper_jaw2_joint"><command_interface name="position"/><state_interface name="position"/><state_interface name="velocity"/></joint> -->
     <joint name="gripper_ABB_Gripper_Finger_1_Joint"><command_interface name="position"/><state_interface name="position"/><state_interface name="velocity"/></joint>
     <joint name="gripper_ABB_Gripper_Finger_2_Joint"><command_interface name="position"/><state_interface name="position"/><state_interface name="velocity"/></joint>

Commit message: fix: gripper in supervisor

File: src/ar4_package/annin_ar4_description/urdf/ar_gripper.ros2_control.xacro (robot description, xacro)
@@ -28,5 +28,5 @@
         </state_interface>
       </joint>
-      <!-- <joint name="${tf_prefix}gripper_jaw2_joint">
+      <joint name="${tf_prefix}gripper_jaw2_joint">
         <param name="mimic">${tf_prefix}gripper_jaw1_joint</param>
         <param name="multiplier">1</param>
@@ -37,5 +37,5 @@
           <param name="initial_value">0.0</param>
         </state_interface>
-      </joint> -->
+      </joint>
     </ros2_control>
   </xacro:macro>
