Commit message: ABB_base_link frame: adjusted the name of the ABB_base_link from Abb_dummy_base

File: src/ar4_package/annin_ar4_driver/urdf/ar.urdf.xacro (robot description, xacro)
@@ -11,9 +11,9 @@
   <xacro:include filename="$(find annin_ar4_description)/urdf/ar_gripper_macro.xacro" />
   <link name="world" />
-  <link name="Abb_dummy_base" />
+  <link name="ABB_base_link" />
   <joint name="ABB_base_joint" type="fixed">
     <parent link="world" />
-    <child link="Abb_dummy_base" />
-    <origin xyz="0 -1.110  0" rpy="0 0 0" />
+    <child link="ABB_base_link" />
+    <origin xyz="0 -1.110  0" rpy="0 0 1.57079" />
   </joint>
   <xacro:ar_robot
