Commit message: feat:launch_file_arguements_added_for_ar4

File: src/dual_arms/urdf/ar4_wrapper.xacro (robot description, xacro)
@@ -1,28 +1,12 @@
 <?xml version="1.0"?>
 <robot xmlns:xacro="http://wiki.ros.org/xacro" name="ar4_robot">
+  <xacro:arg name="ar_model" default="mk3" />
   <xacro:arg name="serial_port" default="/dev/ttyACM0" />
   <xacro:arg name="arduino_serial_port" default="/dev/ttyUSB0" />
-    <!-- CALIBRATE VALUE -->
   <xacro:arg name="calibrate" default="True" />
-    <!--  -->
   <xacro:arg name="tf_prefix" default="ar4_" />
-  <!-- <xacro:arg name="include_gripper" default="False" /> -->
   <xacro:include filename="$(find annin_ar4_description)/urdf/ar.ros2_control.xacro" />
   <xacro:include filename="$(find annin_ar4_description)/urdf/ar_macro.xacro" />
-  <!-- <xacro:include filename="$(find annin_ar4_description)/urdf/ar_gripper.ros2_control.xacro" />
-  <xacro:include filename="$(find annin_ar4_description)/urdf/ar_gripper_macro.xacro" /> -->
-  <!-- <joint name="ABB_base_joint" type="fixed">
-    <parent link="world" />
-    <child link="Abb_dummy_base" />
-    <origin xyz="0 -1.110  0" rpy="0 0 0" />
-  </joint> -->
-  <!-- <xacro:ar_robot
-    tf_prefix="$(arg tf_prefix)"
-    parent="world"
-    robot_parameters_file="$(find annin_ar4_description)/config/mk3.yaml"
-  >
-    <origin xyz="0 0 0" rpy="0 0 0" />
-  </xacro:ar_robot> -->
-  <!-- <xacro:ar_ros2_control
+  <xacro:ar_ros2_control
     ar_model="$(arg ar_model)"
     plugin_name="annin_ar4_driver/ARHardwareInterface"
@@ -33,27 +17,4 @@
     driver_parameters_file="$(find annin_ar4_driver)/config/driver.yaml"
     tf_prefix="$(arg tf_prefix)"
-  /> -->
-  <xacro:ar_ros2_control
-    ar_model="mk3"
-    plugin_name="annin_ar4_driver/ARHardwareInterface"
-    serial_port="$(arg serial_port)"
-    calibrate="$(arg calibrate)"
-    robot_parameters_file="$(find annin_ar4_description)/config/mk3.yaml"
-    joint_offset_parameters_file="$(find annin_ar4_driver)/config/joint_offsets/mk3.yaml"
-    driver_parameters_file="$(find annin_ar4_driver)/config/driver.yaml"
-    tf_prefix="ar4_"
   />
-  <!-- <xacro:if value="$(arg include_gripper)">
-    <xacro:ar_gripper
-      tf_prefix="$(arg tf_prefix)"
-      parent="$(arg tf_prefix)ee_link"
-    />
-    <xacro:ar_gripper_ros2_control
-      name="ar_servo_gripper"
-      plugin_name="annin_ar4_driver/ARServoGripperHWInterface"
-      serial_port="$(arg arduino_serial_port)"
-      driver_parameters_file="$(find annin_ar4_driver)/config/gripper_driver.yaml"
-      tf_prefix="$(arg tf_prefix)"
-    />
-  </xacro:if> -->
 </robot>

File: src/dual_arms/urdf/dual_arms_hardware.xacro (robot description, xacro)
@@ -2,4 +2,10 @@
 <robot name="dual_arms_with_environment" xmlns:xacro="http://www.ros.org/wiki/xacro">
   <xacro:arg name="CONFIG" default="ABB"/>
+  <xacro:arg name="ar_model" default="mk3"/>
+  <xacro:arg name="serial_port" default="/dev/ttyACM0"/>
+  <xacro:arg name="calibrate" default="True"/>
+  <xacro:arg name="tf_prefix" default="ar4_"/>
+  <xacro:arg name="include_gripper" default="True"/>
+  <xacro:arg name="arduino_serial_port" default="/dev/ttyUSB0"/>
   <xacro:include filename="$(find assembly_environment)/urdf/environment_hardware.xacro" />
   <link name="world"/>
@@ -11,20 +17,13 @@
   </joint>
   <xacro:include filename="$(find dual_arms)/urdf/irb120_wrapper.xacro" />
-  <!-- <xacro:include filename="$(find abb_gripper_urdf)/urdf/abb_gripper_macro.xacro" /> -->
   <xacro:irb120_mounted parent="abb_table">
     <origin xyz="0 0 0" rpy="0 0 0"/>
   </xacro:irb120_mounted>
-  <!-- <xacro:abb_gripper arm_parent_link="tool0" gripper_prefix="gripper_"/> -->
-<!-- <xacro:if value="${xacro.arg('CONFIG') != 'ABB'}"> -->
   <xacro:include filename="$(find dual_arms)/urdf/ar4_wrapper.xacro" />
   <xacro:ar_robot
-    tf_prefix="ar4_"
+    tf_prefix="$(arg tf_prefix)"
     parent="ar4_table"
-    robot_parameters_file="$(find annin_ar4_description)/config/mk3.yaml">
+    robot_parameters_file="$(find annin_ar4_description)/config/$(arg ar_model).yaml">
     <origin xyz="0 0 0" rpy="0 0 1.5708"/>
   </xacro:ar_robot>
-  <!-- <xacro:ar_gripper
-    tf_prefix="ar4_"
-    parent="ar4_ee_link"/> -->
-<!-- </xacro:if> -->
 </robot>
